Commit message: Updated wheelchair height and corresponding joint positions

File: urdf/wheelchair_description.xacro (robot description, xacro)
@@ -4,5 +4,6 @@
   <xacro:property name="chair_width" value="0.643" /> <!-- From front wheel right joint to front wheel left joint -->
   <xacro:property name="chair_length" value="0.812" /> <!-- From front wheel joint to back wheel joint -->
-  <xacro:property name="chair_height" value="1.191" /> <!-- From front wheel joint to head rest -->
+  <!-- <xacro:property name="chair_height" value="1.191" /> --> <!-- From front wheel joint to head rest -->
+  <xacro:property name="chair_height" value="0.4" /> <!-- From front wheel joint to approx height -->
   <xacro:property name="chair_weight" value="10.0" />
   <xacro:property name="main_wheel_length" value="0.065" />
@@ -27,5 +28,6 @@
   </link>
   <joint name="base_footprint_joint" type="fixed">
-    <origin xyz=" 0 0 0.7" rpy="0 0 0"/>
+    <!-- <origin xyz=" 0 0 0.7" rpy="0 0 0"/> -->
+    <origin xyz=" 0 0 0.3" rpy="0 0 0"/> <!-- accomodating for change in chair height -->
     <parent link="base_footprint"/>
     <child link="base_link"/>
@@ -125,5 +127,6 @@
     <parent link="right_bar"/>
     <child link="right_main_wheel"/>
-    <origin rpy="1.57075 0 0" xyz="0.0 0.0 -${chair_height/8-0.076}"/>
+    <!-- <origin rpy="1.57075 0 0" xyz="0.0 0.0 -${chair_height/8-0.076}"/> -->
+    <origin rpy="1.57075 0 0" xyz="0.0 0.0 0.026"/> <!-- accomodating for change in chair height -->
   </joint>
   <link name="right_main_wheel">
@@ -150,5 +153,6 @@
     <parent link="left_bar"/>
     <child link="left_main_wheel"/>
-    <origin rpy="1.57075 0 0" xyz="0.0 0.0 -${chair_height/8-0.076}"/>
+    <!-- <origin rpy="1.57075 0 0" xyz="0.0 0.0 -${chair_height/8-0.076}"/> -->
+    <origin rpy="1.57075 0 0" xyz="0.0 0.0 0.026"/> <!-- accomodating for change in chair height -->
   </joint>
   <link name="left_main_wheel">

Commit message: Added Kinect and depth image to laser scan node

File: urdf/wheelchair_description.xacro (robot description, xacro)
@@ -1,5 +1,7 @@
 <?xml version="1.0"?>
 <robot xmlns:xacro="http://www.ros.org/wiki/xacro" name="wheelchair">
+  <xacro:include filename="$(find baxter_wheelchair_description)/urdf/sensors/kinect_camera.urdf.xacro" />
   <xacro:property name="PI" value="3.14159265359" />
+  <xacro:property name="M_PI" value="3.1415926535897931" />
   <xacro:property name="chair_width" value="0.643" /> <!-- From front wheel right joint to front wheel left joint -->
   <xacro:property name="chair_length" value="0.812" /> <!-- From front wheel joint to back wheel joint -->
@@ -13,4 +15,11 @@
   <xacro:property name="small_wheel_length" value=".05" />
   <xacro:property name="small_wheel_weight" value="1.0" />
+  <!-- Kinect Camera Location (Nominally 0) -->
+  <xacro:property name="cal_kinect_x" value="0.0" />
+  <xacro:property name="cal_kinect_y" value="0.0" />
+  <xacro:property name="cal_kinect_z" value="0.0" />
+  <xacro:property name="cal_kinect_roll" value="0.0" />
+  <xacro:property name="cal_kinect_pitch" value="0.0" />
+  <xacro:property name="cal_kinect_yaw" value="0.0" />
   <xacro:macro name="box_intertia" params="height length width weight" >
     <inertia ixx="${1/12 * weight * (height + length)}" ixy="0" ixz="0" iyy="${1/12 * weight * (width + length)}" iyz="0" izz="${1/12 * weight * (width + height)}" />
@@ -52,4 +61,8 @@
     </inertial>
   </link>
+  <!-- Base of Kinect Mount -->
+  <xacro:kinect_camera_v0 name="kinect_camera" parent="base_link" >
+    <origin xyz="${chair_length/2 - 0.02} 0 ${chair_height/2 + 0.05}" rpy="0 0 0" />
+  </xacro:kinect_camera_v0>
   <link name="imu_link">
     <inertial>
