Commit message: Updated wheelchair height

File: urdf/baxter_wheelchair.urdf.xacro (robot description, xacro)
@@ -8,7 +8,9 @@
     <xacro:arg name="gazebo" value="${gazebo}"/>
   </xacro:include>
+  <!-- <xacro:property name="chair_height" value="1.191" /> --> <!-- From front wheel joint to head rest -->
+  <xacro:property name="chair_height" value="0.7" /> <!-- From front wheel joint to approx height -->
   <!-- Link Baxter Base to Wheelchair -->
   <joint name="wheelchair_to_baxter" type="fixed">
-    <origin rpy="0 0 0" xyz="0 0 0.25" />
+    <origin rpy="0 0 0" xyz="0 0 ${chair_height/2 + 0.05}" />
     <parent link="base_link" />
     <child link="base" />

File: urdf/wheelchair_description.xacro (robot description, xacro)
@@ -7,5 +7,5 @@
   <xacro:property name="chair_length" value="0.812" /> <!-- From front wheel joint to back wheel joint -->
   <!-- <xacro:property name="chair_height" value="1.191" /> --> <!-- From front wheel joint to head rest -->
-  <xacro:property name="chair_height" value="0.4" /> <!-- From front wheel joint to approx height -->
+  <xacro:property name="chair_height" value="0.7" /> <!-- From front wheel joint to approx height -->
   <xacro:property name="chair_weight" value="10.0" />
   <xacro:property name="main_wheel_length" value="0.065" />
@@ -38,5 +38,5 @@
   <joint name="base_footprint_joint" type="fixed">
     <!-- <origin xyz=" 0 0 0.7" rpy="0 0 0"/> -->
-    <origin xyz=" 0 0 0.3" rpy="0 0 0"/> <!-- accomodating for change in chair height -->
+    <origin xyz=" 0 0 0.45" rpy="0 0 0"/> <!-- accomodating for change in chair height -->
     <parent link="base_footprint"/>
     <child link="base_link"/>
@@ -141,5 +141,5 @@
     <child link="right_main_wheel"/>
     <!-- <origin rpy="1.57075 0 0" xyz="0.0 0.0 -${chair_height/8-0.076}"/> -->
-    <origin rpy="1.57075 0 0" xyz="0.0 0.0 0.026"/> <!-- accomodating for change in chair height -->
+    <origin rpy="1.57075 0 0" xyz="0.0 0.0 ${main_wheel_radius - chair_height/8 - small_wheel_radius}"/> <!-- accomodating for change in chair height -->
   </joint>
   <link name="right_main_wheel">
@@ -167,5 +167,5 @@
     <child link="left_main_wheel"/>
     <!-- <origin rpy="1.57075 0 0" xyz="0.0 0.0 -${chair_height/8-0.076}"/> -->
-    <origin rpy="1.57075 0 0" xyz="0.0 0.0 0.026"/> <!-- accomodating for change in chair height -->
+    <origin rpy="1.57075 0 0" xyz="0.0 0.0 ${main_wheel_radius - chair_height/8 - small_wheel_radius}"/> <!-- accomodating for change in chair height -->
   </joint>
   <link name="left_main_wheel">

Commit message: Reverted to chair height 0.4

File: urdf/baxter_wheelchair.urdf.xacro (robot description, xacro)
@@ -9,5 +9,5 @@
   </xacro:include>
   <!-- <xacro:property name="chair_height" value="1.191" /> --> <!-- From front wheel joint to head rest -->
-  <xacro:property name="chair_height" value="0.7" /> <!-- From front wheel joint to approx height -->
+  <xacro:property name="chair_height" value="0.4" /> <!-- From front wheel joint to approx height -->
   <!-- Link Baxter Base to Wheelchair -->
   <joint name="wheelchair_to_baxter" type="fixed">

File: urdf/wheelchair_description.xacro (robot description, xacro)
@@ -7,5 +7,5 @@
   <xacro:property name="chair_length" value="0.812" /> <!-- From front wheel joint to back wheel joint -->
   <!-- <xacro:property name="chair_height" value="1.191" /> --> <!-- From front wheel joint to head rest -->
-  <xacro:property name="chair_height" value="0.7" /> <!-- From front wheel joint to approx height -->
+  <xacro:property name="chair_height" value="0.4" /> <!-- From front wheel joint to approx height -->
   <xacro:property name="chair_weight" value="10.0" />
   <xacro:property name="main_wheel_length" value="0.065" />
@@ -38,5 +38,5 @@
   <joint name="base_footprint_joint" type="fixed">
     <!-- <origin xyz=" 0 0 0.7" rpy="0 0 0"/> -->
-    <origin xyz=" 0 0 0.45" rpy="0 0 0"/> <!-- accomodating for change in chair height -->
+    <origin xyz=" 0 0 0.3" rpy="0 0 0"/> <!-- accomodating for change in chair height -->
     <parent link="base_footprint"/>
     <child link="base_link"/>

Commit message: Updated position of baxter on wheelchair to make it more stable

File: urdf/baxter_wheelchair.urdf.xacro (robot description, xacro)
@@ -12,5 +12,5 @@
   <!-- Link Baxter Base to Wheelchair -->
   <joint name="wheelchair_to_baxter" type="fixed">
-    <origin rpy="0 0 0" xyz="0 0 ${chair_height/2 + 0.05}" />
+    <origin rpy="0 0 0" xyz="-0.1 0 ${chair_height/2 + 0.05}" />
     <parent link="base_link" />
     <child link="base" />
